File: Electronics/Motherboard/CurrentVersion/motherboard_2layers_v2.kicad_pcb (KiCad board)
At the start: 2 copper layers, 113.4 x 56 mm, 87 parts, among them J1 Conn_02x10_Odd_Even, J2 SSD1306, J3 USB_C_Receptacle_USB2.0_16P, J4 Micro_SD_Card_Det2, J5 Encoder, Q1 FDMS86202, Q2 FDMS86202, Q3 AO3400A, Q4 AO3400A, Q5 AO3400A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

Commit message: Finished layout
Parts:
- removed the R8 at (69.9, 130.3)
- removed the R8 at (240.0, 148.2)
- added R8: 4.7k, Resistor_SMD:R_1206_3216Metric, F.Cu at (172.8, 66.2)
- added SW1: ~, ad-hoc:ALPSALPINE_TopPush_Button, F.Cu at (196.9, 71.7)
- J2: footprint Connector_PinHeader_2.54mm:PinHeader_1x04_P2.54mm_Vertical -> Connector_JST:JST_XH_B4B-XH-A_1x04_P2.50mm_Vertical
- moved C24 218.7 mm to (218.6, 58.6)
- moved R11 203.8 mm to (215.8, 74.2), turned to -90 degrees
- moved C23 203.6 mm to (211.8, 73.3), turned to -90 degrees
- moved U9 158.6 mm to (223.8, 51.6), turned to 180 degrees
- moved C26 155.5 mm to (219.1, 38.8), turned to -90 degrees
- moved R10 150.3 mm to (227.8, 51.2), turned to -90 degrees
- moved C27 149.3 mm to (210.7, 38.8), turned to -90 degrees
- moved R9 147.5 mm to (228.6, 56.2), turned to 90 degrees
- moved C28 143.3 mm to (202.2, 38.8), turned to -90 degrees
- moved R1 139.6 mm to (216.2, 70.1), turned to 90 degrees
- moved R2 137.6 mm to (183.8, 69.7), turned to -90 degrees
- moved C19 136.4 mm to (201.9, 61.3), turned to 90 degrees
- moved R3 132.4 mm to (180.1, 69.7), turned to -90 degrees
- moved J1 131.8 mm to (211.5, 45.5), turned to 90 degrees
- moved C1 128.0 mm to (197.8, 59.6)
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Connections:
- net Net-(J3-D+-PadA6) renamed /RAW_D+
- net Net-(J3-D--PadA7) renamed /RAW_D-
- J3 pad A4: +5V -> VBUS
- J3 pad A9: +5V -> VBUS
- J3 pad B4: +5V -> VBUS
- J3 pad B9: +5V -> VBUS
- U9 pad 5: +5V -> VBUS
Other:
- board size 113.4 x 56 mm -> 113.4 x 71.2 mm
