File: Electronics/Motherboard/CurrentVersion/motherboard_2layers_v2.kicad_sch (KiCad schematic)
At the start: 87 parts, among them J1 Conn_02x10_Odd_Even, J2 SSD1306, J3 USB_C_Receptacle_USB2.0_16P, J4 Micro_SD_Card_Det2, J5 Encoder, Q1 FDMS86202, Q2 FDMS86202, Q3 AO3400A, Q4 AO3400A, Q5 AO3400A, SW1 SW_Push, U1 TMC2209_SilentStepStick, U2 TMC2209_SilentStepStick, U3 LY1576HVS-5, U4 TMC2209_SilentStepStick, U5 TMC2209_SilentStepStick, U6 STZ12F405RGTx, U7 AMS1117-3.3, U8 AW9523B, U9 USBLC6-2SC6

Commit message: aaaaaa many new thingies
Parts:
- C10, C11, C12, C13, C14, C15, C16, C17, C18, C3, C4, C5, C6, C7, C8, C9: footprint Capacitor_SMD:C_0402_1005Metric -> Capacitor_SMD:C_0201_0603Metric; Part # TCC0402X7R104K160AT -> GRM033R61A104KE15D
- FAN1, FAN2, FAN3: footprint ad-hoc:ScrewTerminal-2pin-MKDS_1_2-3_5 -> Connector_JST:JST_XH_B2B-XH-A_1x02_P2.50mm_Vertical
- U8: footprint Package_DFN_QFN:QFN-24-1EP_4x4mm_P0.5mm_EP2.7x2.7mm_ThermalVias -> Package_DFN_QFN:QFN-24-1EP_4x4mm_P0.5mm_EP2.7x2.7mm
Connections:
- net at U5.3 (M1B): now also MOTOR_E1.4 (Pin_4); no longer MOTOR_E1.3 (Pin_3)
- net at U5.4 (M1A): now also MOTOR_E1.3 (Pin_3); no longer MOTOR_E1.1 (Pin_1)
- net at U5.6 (M2B): now also MOTOR_E1.1 (Pin_1); no longer MOTOR_E1.4 (Pin_4)
- net at U2.3 (M1B): now also MOTOR_Y1.4 (Pin_4); no longer MOTOR_Y1.3 (Pin_3)
- net at U2.4 (M1A): now also MOTOR_Y1.3 (Pin_3); no longer MOTOR_Y1.1 (Pin_1)
- net at U2.6 (M2B): now also MOTOR_Y1.1 (Pin_1); no longer MOTOR_Y1.4 (Pin_4)
- net at U4.3 (M1B): now also MOTOR_Z1.4 (Pin_4); no longer MOTOR_Z1.3 (Pin_3)
- net at U4.4 (M1A): now also MOTOR_Z1.3 (Pin_3); no longer MOTOR_Z1.1 (Pin_1)
- net at U4.6 (M2B): now also MOTOR_Z1.1 (Pin_1); no longer MOTOR_Z1.4 (Pin_4)
- net at MOTOR_X1.1 (Pin_1): now also U1.6 (M2B); no longer U1.4 (M1A)
- net at MOTOR_X1.3 (Pin_3): now also U1.4 (M1A); no longer U1.3 (M1B)
- net at MOTOR_X1.4 (Pin_4): now also U1.3 (M1B); no longer U1.6 (M2B)
Other:
- moved on the sheet: MOTOR_X1

Commit message: Finished layout
Parts:
- F1: footprint RUEF900:FUSRR1015W81L2410T300H2900 -> ad-hoc:Fuse_RUEF900
- J2: footprint Connector_PinHeader_2.54mm:PinHeader_1x04_P2.54mm_Vertical -> Connector_JST:JST_XH_B4B-XH-A_1x04_P2.50mm_Vertical
- JP1: footprint (none) -> TestPoint:TestPoint_2Pads_Pitch2.54mm_Drill0.8mm; now left out of the parts list
- R10, R9: footprint RMCF0805JT5K10:RESC2012X65N -> Resistor_SMD:R_0805_2012Metric; Part # (none) -> RMCF0805JT5K10
- R8: Part # RC1206JR-134K7L -> (none)
- SW1: value SW_Push -> ~; footprint (none) -> ad-hoc:ALPSALPINE_TopPush_Button; Part # (none) -> SKHHAMA010
Connections:
- net +5V: no longer J3.A4 (VBUS), J3.A9 (VBUS), J3.B4 (VBUS), J3.B9 (VBUS), U9.5 (VBUS)
- net EN_BTN: now also R8.2; no longer R8.1
- net GND: now also R8.1; no longer R8.2
- net RAW_D-: now reaches J3.A7 (D-), J3.B7 (D-), U9.1 (I/O1)
- net RAW_D+: now reaches J3.A6 (D+), J3.B6 (D+), U9.3 (I/O2)
- new net VBUS: J3.A4 (VBUS), J3.A9 (VBUS), J3.B4 (VBUS), J3.B9 (VBUS), U9.5 (VBUS)
