File: Electronics/Motherboard/CurrentVersion/Motherboard2.4 (small)/motherboard_2layers_v2.kicad_pcb (KiCad board)
At the start: 2 copper layers, 113.4 x 71.2 mm, 87 parts, among them J1 Conn_02x10_Odd_Even, J2 SSD1306, J3 USB_C_Receptacle_USB2.0_16P, J4 Micro_SD_Card_Det2, J5 Encoder, Q1 FDMS86202, Q2 FDMS86202, Q3 AO3400A, Q4 AO3400A, Q5 AO3400A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

Commit message: tinny pcb
Parts:
- C23, C24: footprint Capacitor_SMD:C_1206_3216Metric -> Capacitor_SMD:C_0603_1608Metric
- D1: footprint Diode_THT:D_DO-201AD_P15.24mm_Horizontal -> Diode_SMD:D_SOD-123
- R10, R9: footprint Resistor_SMD:R_0805_2012Metric -> Resistor_SMD:R_0402_1005Metric
- R11, R2, R3: footprint Resistor_SMD:R_1206_3216Metric -> Resistor_SMD:R_0603_1608Metric
- moved R4 60.1 mm to (164.9, 52.0)
- moved THM1 60.1 mm to (165.1, 45.1)
- moved C26 58.8 mm to (161.8, 52.0), turned to 90 degrees
- moved J1 49.5 mm to (163.8, 58.5)
- moved J5 46.5 mm to (215.5, 30.8)
- moved THM2 44.0 mm to (173.4, 45.2)
- moved R6 43.7 mm to (173.4, 52.0)
- moved C27 42.4 mm to (170.4, 52.0), turned to 90 degrees
- moved R11 40.2 mm to (193.8, 40.6), turned to 90 degrees
- moved J4 39.7 mm to (202.6, 36.6), turned to 180 degrees
- moved SW1 35.2 mm to (221.4, 46.4)
- moved D3 34.7 mm to (151.2, 54.2)
- moved R8 32.0 mm to (189.0, 38.6)
- moved THM3 28.7 mm to (181.6, 45.2)
- moved R7 28.1 mm to (182.0, 52.0)
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Other:
- board size 113.4 x 71.2 mm -> 113.4 x 55.3 mm

Commit message: Started routing
Parts:
- moved R8 41.7 mm to (230.1, 31.4), turned to 90 degrees
- moved R9 6.14 mm to (227.9, 42.1)
- moved R10 4.68 mm to (227.8, 37.1), turned to -90 degrees
- moved R3 2.09 mm to (168.8, 63.5), turned to 180 degrees
- moved R2 1.69 mm to (169.5, 65.3), turned to 180 degrees
- moved D1 0.55 mm to (148.4, 48.4), turned to -90 degrees
- moved U9 0.28 mm to (213.5, 45.0), turned to 180 degrees
- turned F1 to 0 degrees
Connections:
- net USB_DM renamed USB_D-
- net USB_DP renamed USB_D+
Routing:
- net GND: track 0.00 -> 392.4 mm
- net +3V3: track 0.00 -> 209.3 mm, vias 0 -> 3
- net +24V: track 0.00 -> 160.4 mm, vias 0 -> 1
- net +5V: track 0.00 -> 117.2 mm
- net NEOPIXEL_DIN: track 0.00 -> 89.2 mm, vias 0 -> 4
- net Net-(D3-DOUT): track 0.00 -> 88.7 mm, vias 0 -> 2
- net BED: track 0.00 -> 76.1 mm, vias 0 -> 2
- net HOTEND: track 0.00 -> 73.4 mm, vias 0 -> 2
- net /RAW_D-: track 0.00 -> 36.3 mm, vias 0 -> 2
- net /RAW_D+: track 0.00 -> 36.0 mm, vias 0 -> 2
- net VBUS: track 0.00 -> 29.0 mm, vias 0 -> 2
- net Net-(D2-DOUT): track 0.00 -> 27.6 mm
- net Net-(D1-K): track 0.00 -> 17.3 mm
- net SD_CONN: track 0.00 -> 16.4 mm
- net EN_BTN: track 0.00 -> 13.5 mm
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- added copper zone on B.Cu, net GND
- added copper zone on F.Cu, net GND

Commit message: Did some routing
Parts:
- moved C25 0.56 mm to (168.7, 61.8)
- moved R3 0.56 mm to (169.2, 63.1)
- moved R2 0.56 mm to (169.8, 64.9)
- turned R1 to 180 degrees
Routing:
- net DIR_E1: track 0.00 -> 108.3 mm, vias 0 -> 3
- net EN_E1: track 0.00 -> 93.9 mm, vias 0 -> 1
- net DIAG_E1: track 0.00 -> 87.8 mm, vias 0 -> 3
- net DRIVER_UART: track 0.00 -> 83.8 mm
- net STEP_E1: track 0.00 -> 67.8 mm, vias 0 -> 1
- net INDEX_E1: track 0.00 -> 66.9 mm, vias 0 -> 2
- net +3V3: track 209.3 -> 271.1 mm, vias 3 -> 7
- net STEP_Z1: track 0.00 -> 55.8 mm, vias 0 -> 1
- net +24V: track 160.4 -> 215.4 mm, vias 1 -> 2
- net DIAG_Z1: track 0.00 -> 49.0 mm, vias 0 -> 4
- net EN_FOR: track 0.00 -> 48.4 mm, vias 0 -> 1
- net SCRN_SCL: track 0.00 -> 45.7 mm, vias 0 -> 6
- net EN_Z1: track 0.00 -> 42.3 mm, vias 0 -> 1
- net FAN1: track 0.00 -> 40.9 mm, vias 0 -> 2
- net SCRN_SDA: track 0.00 -> 39.9 mm, vias 0 -> 4
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
Commit message: Fixed a typo that's been there for idk how long
Parts:
- turned BED1 to 180 degrees
- turned HOTEND1 to 180 degrees
Routing:
- net +5V: track 116.6 -> 190.3 mm, vias 0 -> 1
- net +24V: track 215.4 -> 226.2 mm
- net Net-(HOTEND1-Pin_1): track 8.48 -> 11.0 mm
- net Net-(BED1-Pin_1): track 8.30 -> 10.7 mm
- net HOTEND: track 75.4 -> 73.8 mm
